File: Technology/ARBO Testbed/ARBO Testbed.sch (KiCad schematic (older format))
At the start: 88 parts, among them J1 USB_B_Micro, J2 Micro_SD_Card_473093351, J3 IN1, J4 IN2, J5 IN3, J6 BIAS, J7 IN4, SW1 SW_SPST, U1 MCP73831-2-OT, U2 MAX828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

Commit message: Updating values to match changes on board
Parts:
- added TP?: TP_SWCLK, TestPoint:TestPoint_THTPad_3.0x3.0mm_Drill1.5mm, symbol Connector:TestPoint
- added TP?: TP_SWDIO, TestPoint:TestPoint_THTPad_3.0x3.0mm_Drill1.5mm, symbol Connector:TestPoint
- C2, C3: value 1uF -> 22pF
- R2, R6: value 1K -> 2.2K
Connections:
- net at U6.45 (PA30): now also TP?.1
- net at U6.46 (PA31): now also TP?.1
- no-connect marks 16 -> 14
Other:
- moved on the sheet: SW1
Changed lines of the file:
@@
 P 1750 1900
 F 0 "R2" V 1543 1900 50  0000 C CNN
-F 1 "1K" V 1634 1900 50  0000 C CNN
+F 1 "2.2K" V 1634 1900 50  0000 C CNN
 F 2 "Resistor_SMD:R_0603_1608Metric" V 1680 1900 50  0001 C CNN
 F 3 "~" H 1750 1900 50  0001 C CNN
@@
 P 8250 2100
 F 0 "R6" H 8180 2054 50  0000 R CNN
-F 1 "1K" H 8180 2145 50  0000 R CNN
+F 1 "2.2K" H 8180 2145 50  0000 R CNN
 F 2 "Resistor_SMD:R_0603_1608Metric" V 8180 2100 50  0001 C CNN
 F 3 "~" H 8250 2100 50  0001 C CNN
@@
 $EndComp
 $Comp
-L Device:R R7
-U 1 1 5DF17EA3
-P 8650 2100
-F 0 "R7" H 8580 2054 50  0000 R CNN
-F 1 "2.2K" H 8580 2145 50  0000 R CNN
-F 2 "Resistor_SMD:R_0603_1608Metric" V 8580 2100 50  0001 C CNN
-F 3 "~" H 8650 2100 50  0001 C CNN
-F 4 "P2.2KGCT-ND" H 8650 2100 50  0001 C CNN "Digi-key Part Number"
-F 5 "ERJ-3GEYJ222V" H 8650 2100 50  0001 C CNN "Manufacturer Part Number"
-	1    8650 2100
-	-1   0    0    1
-$EndComp
-$Comp
 L power:GNDD #PWR09
 U 1 1 5DF17EA9
@@
 P 12700 950
 F 0 "C3" H 12600 1050 50  0000 L CNN
-F 1 "1uF" H 12500 850 50  0000 L CNN
+F 1 "22pF" H 12500 850 50  0000 L CNN
 F 2 "Capacitor_SMD:C_0402_1005Metric" H 12738 800 50  0001 C CNN
 F 3 "~" H 12700 950 50  0001 C CNN
@@
 P 12400 950
 F 0 "C2" H 12300 1050 50  0000 L CNN
-F 1 "1uF" H 12200 850 50  0000 L CNN
+F 1 "22pF" H 12200 850 50  0000 L CNN
 F 2 "Capacitor_SMD:C_0402_1005Metric" H 12438 800 50  0001 C CNN
 F 3 "~" H 12400 950 50  0001 C CNN
@@
 Wire Wire Line
 	4400 1950 4400 1900
-$Comp
-L Device:R R4
-U 1 1 5DFFBB13
-P 4400 2100
-F 0 "R4" H 4470 2146 50  0000 L CNN
-F 1 "10K" H 4470 2055 50  0000 L CNN
-F 2 "Resistor_SMD:R_0603_1608Metric" V 4330 2100 50  0001 C CNN
-F 3 "~" H 4400 2100 50  0001 C CNN
-F 4 "311-10KGRCT-ND" H 4400 2100 50  0001 C CNN "Digi-key Part Number"
-F 5 "RC0603JR-0710KL" H 4400 2100 50  0001 C CNN "Manufacturer Part Number"
-	1    4400 2100
-	1    0    0    -1
-$EndComp
 Text GLabel 4950 2000 0    50   Input ~ 0
 ~EC_PWDN
 NoConn ~ 12800 4000
 NoConn ~ 12800 4100
-NoConn ~ 12800 4200
-NoConn ~ 12800 4300
 NoConn ~ 14800 1500
 NoConn ~ 14800 2000
@@
 L Switch:SW_SPST SW1
 U 1 1 5E07945F
-P 12450 4500
-F 0 "SW1" H 12450 4275 50  0000 C CNN
-F 1 "SW_SPST" H 12450 4366 50  0000 C CNN
-F 2 "Button_Switch_SMD:SW_SPST_PTS810" H 12450 4500 50  0001 C CNN
-F 3 "~" H 12450 4500 50  0001 C CNN
-F 4 "CKN10503TR-ND" H 12450 4500 50  0001 C CNN "Digi-key Part Number"
-F 5 "PTS810 SJK 250 SMTR LFS" H 12450 4500 50  0001 C CNN "Manufacturer Part Number"
-	1    12450 4500
+P 11400 4500
+F 0 "SW1" H 11400 4275 50  0000 C CNN
+F 1 "SW_SPST" H 11400 4366 50  0000 C CNN
+F 2 "Button_Switch_SMD:SW_SPST_PTS810" H 11400 4500 50  0001 C CNN
+F 3 "~" H 11400 4500 50  0001 C CNN
+F 4 "CKN10503TR-ND" H 11400 4500 50  0001 C CNN "Digi-key Part Number"
+F 5 "PTS810 SJK 250 SMTR LFS" H 11400 4500 50  0001 C CNN "Manufacturer Part Number"
+	1    11400 4500
 	-1   0    0    1
 $EndComp
@@
 L power:GNDD #PWR014
 U 1 1 5E07BB78
-P 12250 4600
-F 0 "#PWR014" H 12250 4350 50  0001 C CNN
-F 1 "GNDD" H 12254 4445 50  0000 C CNN
-F 2 "" H 12250 4600 50  0001 C CNN
-F 3 "" H 12250 4600 50  0001 C CNN
-	1    12250 4600
-	1    0    0    -1
-$EndComp
-Wire Wire Line
-	12250 4500 12250 4600
-Wire Wire Line
-	12650 4500 12800 4500
+P 11200 4600
+F 0 "#PWR014" H 11200 4350 50  0001 C CNN
+F 1 "GNDD" H 11204 4445 50  0000 C CNN
+F 2 "" H 11200 4600 50  0001 C CNN
+F 3 "" H 11200 4600 50  0001 C CNN
+	1    11200 4600
+	1    0    0    -1
+$EndComp
+Wire Wire Line
+	11200 4500 11200 4600
 $Comp
 L Device:C C15
@@
 Text GLabel 14800 1700 2    50   Input ~ 0
 A2
+$Comp
+L Device:R R4
+U 1 1 5DFFBB13
+P 4400 2100
+F 0 "R4" H 4470 2146 50  0000 L CNN
+F 1 "10K" H 4470 2055 50  0000 L CNN
+F 2 "Resistor_SMD:R_0603_1608Metric" V 4330 2100 50  0001 C CNN
+F 3 "~" H 4400 2100 50  0001 C CNN
+F 4 "311-10KGRCT-ND" H 4400 2100 50  0001 C CNN "Digi-key Part Number"
+F 5 "RC0603JR-0710KL" H 4400 2100 50  0001 C CNN "Manufacturer Part Number"
+	1    4400 2100
+	1    0    0    -1
+$EndComp
+$Comp
+L Device:R R7
+U 1 1 5DF17EA3
+P 8650 2100
+F 0 "R7" H 8580 2054 50  0000 R CNN
+F 1 "2.2K" H 8580 2145 50  0000 R CNN
+F 2 "Resistor_SMD:R_0603_1608Metric" V 8580 2100 50  0001 C CNN
+F 3 "~" H 8650 2100 50  0001 C CNN
+F 4 "P2.2KGCT-ND" H 8650 2100 50  0001 C CNN "Digi-key Part Number"
+F 5 "ERJ-3GEYJ222V" H 8650 2100 50  0001 C CNN "Manufacturer Part Number"
+	1    8650 2100
+	-1   0    0    1
+$EndComp
+$Comp
+L Connector:TestPoint TP?
+U 1 1 5E148BC4
+P 12350 4200
+F 0 "TP?" H 12408 4318 50  0000 L CNN
+F 1 "TP_SWCLK" H 12408 4227 50  0000 L CNN
+F 2 "TestPoint:TestPoint_THTPad_3.0x3.0mm_Drill1.5mm" H 12550 4200 50  0001 C CNN
+F 3 "~" H 12550 4200 50  0001 C CNN
+F 4 "36-5009-ND" H 12350 4200 50  0001 C CNN "Digi-key Part Number"
+F 5 "5009" H 12350 4200 50  0001 C CNN "Manufacturer Part Number"
+	1    12350 4200
+	1    0    0    -1
+$EndComp
+Wire Wire Line
+	11600 4500 12800 4500
+$Comp
+L Connector:TestPoint TP?
+U 1 1 5E1A747E
+P 12050 4300
+F 0 "TP?" H 12108 4418 50  0000 L CNN
+F 1 "TP_SWDIO" H 12108 4327 50  0000 L CNN
+F 2 "TestPoint:TestPoint_THTPad_3.0x3.0mm_Drill1.5mm" H 12250 4300 50  0001 C CNN
+F 3 "~" H 12250 4300 50  0001 C CNN
+F 4 "36-5009-ND" H 12050 4300 50  0001 C CNN "Digi-key Part Number"
+F 5 "5009" H 12050 4300 50  0001 C CNN "Manufacturer Part Number"
+	1    12050 4300
+	1    0    0    -1
+$EndComp
+Wire Wire Line
+	12350 4200 12800 4200
+Wire Wire Line
+	12050 4300 12800 4300
 $EndSCHEMATC

Commit message: Exported gerbers
Parts:
- U6: symbol MCU_Microchip_SAMD:ATSAMD21G18A-AUT -> ARBO-Testbed-rescue:ATSAMD21G18A-AUT-MCU_Microchip_SAMD
Changed lines of the file:
@@
 	6250 1150 6400 1150
 $Comp
-L MCU_Microchip_SAMD:ATSAMD21G18A-AUT U6
+L ARBO-Testbed-rescue:ATSAMD21G18A-AUT-MCU_Microchip_SAMD U6
 U 1 1 5DE77A6D
 P 13800 3000
