File: Technology/ARBO Mini/ARBO Mini.sch (KiCad schematic (older format))
At the start: 85 parts, among them J1 USB_B_Micro, J2 Micro_SD_Card_473093351, J3 Conn_01x10, SW1 SW_SPST, U1 MCP73831-2-OT, U2 MAX828, U3 ICM-20948, U4 SPX3819M5-L-3-3, U5 MAX1726EUK18+, U6 ATSAMD21G18A-AUT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

Commit message: ARBO mini sent to JSTPCB for fab
Parts:
- added U10: SiT1532, ARBO:SiT1532, symbol ARBO:SiT1532
- C2, C3: Digi-key Part Number 399-4873-1-ND -> 399-7775-1-ND; Manufacturer Part Number C0402C105K9PACTU -> C0402C220K5GACTU
- CONN1: Digi-key Part Number 455-3957-1-ND -> (none); Manufacturer Part Number SM02B-SHLS-TF(LF)(SN) -> (none)
- D3: Digi-key Part Number 160-1447-1-ND -> 732-11991-1-ND; Manufacturer Part Number LTST-C191KRKT -> 150040RS73240
- D4: Digi-key Part Number 160-1445-1-ND -> 732-11991-1-ND; Manufacturer Part Number LTST-C191KFKT -> 150040RS73240
- D5: Digi-key Part Number 160-1447-1-ND -> 732-11992-1-ND; Manufacturer Part Number LTST-C191KRKT -> 150040VS73240
- J3: footprint Connector_Hirose:Hirose_DF52-10S-0.8H_1x10-1MP_P0.80mm_Horizontal -> Connector_Hirose:Hirose_DF52-12S-0.8H_1x12-1MP_P0.80mm_Horizontal; symbol Connector_Generic:Conn_01x10 -> Connector_Generic:Conn_01x12; Digi-key Part Number (none) -> H125103CT-ND; Manufacturer Part Number (none) -> DF52-12S-0.8H(21)
- R1, R5: Digi-key Part Number (none) -> 311-100KLRCT-ND; Manufacturer Part Number (none) -> RC0402FR-07100KL
- R10, R11, R12, R13, R14, R15, R17, R18, R7, R9: Digi-key Part Number (none) -> 311-2.20KLRCT-ND; Manufacturer Part Number ERJ-3GEYJ222V -> RC0402FR-072K2L
- R16: Digi-key Part Number (none) -> 311-1.00MLRCT-ND; Manufacturer Part Number (none) -> RC0402FR-071ML
- R2: Digi-key Part Number (none) -> 311-2.20KLRCT-ND; Manufacturer Part Number RC0603JR-071KL -> RC0402FR-072K2L
- R3, R4, R8: Digi-key Part Number (none) -> 311-10.0KLRCT-ND; Manufacturer Part Number (none) -> RC0402FR-0710KL
- R6: Digi-key Part Number (none) -> 311-0.0JRCT-ND; Manufacturer Part Number (none) -> RC0402JR-070RL
Connections:
- net +3V3: now also U10.3 (Vdd)
- net EC_START: now also U6.25 (PA16/~D11); no longer U6.24 (PA15/~D5)
- net GNDD: now also U10.1 (GND), U10.4 (GND)
- net HI_IN1N: now also J3.11 (Pin_11); no longer J3.9 (Pin_9)
- net HI_IN1P: now also J3.12 (Pin_12); no longer J3.10 (Pin_10)
- net HI_IN2N: now also J3.9 (Pin_9); no longer J3.7 (Pin_7)
- net HI_IN2P: now also J3.10 (Pin_10); no longer J3.8 (Pin_8)
- net HI_IN3N: now also J3.7 (Pin_7); no longer J3.5 (Pin_5)
- net HI_IN3P: now also J3.8 (Pin_8); no longer J3.6 (Pin_6)
- net HI_IN4N: now also J3.5 (Pin_5); no longer J3.3 (Pin_3)
- net HI_IN4P: now also J3.6 (Pin_6); no longer J3.4 (Pin_4)
- net SD_CS: now also U6.24 (PA15/~D5); no longer U6.23 (PA14/D2/XIN)
- new net: U10.2 (CLK_Out), U6.23 (PA14/D2/XIN)
- no-connect marks 28 -> 27
Other:
- moved on the sheet: C11, U3

Commit message: ARBO mini FRAM pads are backwards, fix later
Parts:
- C19: value 0.1uF -> 1uF
Changed lines of the file:
@@
 P 4900 6950
 F 0 "C19" H 4800 7050 50  0000 L CNN
-F 1 "0.1uF" H 4700 6850 50  0000 L CNN
+F 1 "1uF" H 4700 6850 50  0000 L CNN
 F 2 "Capacitor_SMD:C_0402_1005Metric" H 4938 6800 50  0001 C CNN
 F 3 "~" H 4900 6950 50  0001 C CNN
