File: Technology/ESLO_Debugger/ESLO_Debugger.sch (KiCad schematic (older format))
At the start: 14 parts, among them J1 USB_B_Micro, J2 Screw_Terminal_01x02, J3 Conn_01x06_Male, Q1 BSS138, Q2 BSS138, U1 LP5907MFX-1.8

Commit message: Reconsidering ESLO architecture (-> CC2640R2)
Other:
- note added: "See Figure 44-14: it doesn’t show line level being an issue?"
Changed lines of the file:
@@
 	3000 2950 3700 2950
 Connection ~ 2400 2700
+Text Notes 1450 3950 0    50   ~ 0
+See Figure 44-14: it doesn’t show line level being an issue?
 $EndSCHEMATC
