File: Technology/ESLO_PSP/ESLO_PSP.kicad_pcb (KiCad board)
At the start: 2 copper layers, 51.8 x 67.1 mm, 41 parts, among them J1 Imeas, P5 Digital, P6 Analog, U1 LP5907MFX-1.8, U2 LP5907MFX-1.5, U3 MAX1720, U4 TPS72301DDCT, U5 nRF24L01P, U6 AN91445, Y1 SXT21412AA16

Commit message: ESLO project updates
Parts:
- added TP5: TPGNDD, TestPoint:TestPoint_Keystone_5000-5004_Miniature, F.Cu at (147.5, 91.8)
Changed lines of the file:
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@@
     (tracks 299)
     (zones 0)
-    (modules 41)
+    (modules 42)
     (nets 28)
   )
@@
     (uvia_drill 0.1)
     (add_net +1V8)
+    (add_net +3V3)
+    (add_net +5V)
     (add_net +BATT)
+    (add_net "/0(Rx)")
+    (add_net "/1(Tx)")
+    (add_net /4)
+    (add_net "/5(**)")
+    (add_net "/6(**)")
+    (add_net /7)
+    (add_net /8)
+    (add_net "/9(**)")
+    (add_net /A0)
+    (add_net /A1)
+    (add_net /A2)
+    (add_net /A3)
+    (add_net /A4)
+    (add_net /A5)
+    (add_net /A6)
+    (add_net /A7)
+    (add_net /AREF)
+    (add_net /Vin)
     (add_net CE)
     (add_net GNDA)
@@
     (add_net "Net-(L1-Pad1)")
     (add_net "Net-(L2-Pad2)")
+    (add_net "Net-(P5-Pad3)")
+    (add_net "Net-(P6-Pad3)")
     (add_net "Net-(R4-Pad1)")
+    (add_net "Net-(U1-Pad4)")
+    (add_net "Net-(U2-Pad4)")
     (add_net SCK)
     (add_net SS)
@@
   )
   (module TestPoint:TestPoint_Keystone_5000-5004_Miniature (layer F.Cu)
+    (at 147.5 91.75)
+    (descr "Keystone Miniature THM Test Point 5000-5004, http://www.keyelco.com/product-pdf.cfm?p=1309")
+    (tags "Through Hole Mount Test Points")
+    (fp_text reference TP5 (at 0 -2.5) (layer F.SilkS)
+      (effects (font (size 1 1) (thickness 0.15)))
+    )
+    (fp_text value TPGNDD (at 0 2.5) (layer F.Fab)
+      (effects (font (size 1 1) (thickness 0.15)))
+    )
+    (fp_circle (center 0 0) (end 1.4 0) (layer F.SilkS) (width 0.15))
+    (fp_circle (center 0 0) (end 1.25 0) (layer F.Fab) (width 0.15))
+    (fp_circle (center 0 0) (end 1.65 0) (layer F.CrtYd) (width 0.05))
+    (fp_line (start -0.75 0.25) (end -0.75 -0.25) (layer F.Fab) (width 0.15))
+    (fp_line (start 0.75 0.25) (end -0.75 0.25) (layer F.Fab) (width 0.15))
+    (fp_line (start 0.75 -0.25) (end 0.75 0.25) (layer F.Fab) (width 0.15))
+    (fp_line (start -0.75 -0.25) (end 0.75 -0.25) (layer F.Fab) (width 0.15))
+    (fp_text user %R (at 0 -2.5) (layer F.Fab)
+      (effects (font (size 1 1) (thickness 0.15)))
+    )
+    (pad 1 thru_hole circle (at 0 0) (size 2 2) (drill 1) (layers *.Cu *.Mask)
+      (net 5 GNDD))
+    (model ${KISYS3DMOD}/TestPoint.3dshapes/TestPoint_Keystone_5000-5004_Miniature.wrl
+      (at (xyz 0 0 0))
+      (scale (xyz 1 1 1))
+      (rotate (xyz 0 0 0))
+    )
+  )
+  (module TestPoint:TestPoint_Keystone_5000-5004_Miniature (layer F.Cu)

Commit message: Reconsidering ESLO architecture (-> CC2640R2)
Parts:
- C4, C5: value 1uF -> 10uF
Connections:
- TP5 pad 1: GNDD -> GNDA
Changed lines of the file:
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@@
     )
     (pad 1 thru_hole circle (at 0 0) (size 2 2) (drill 1) (layers *.Cu *.Mask)
-      (net 5 GNDD))
+      (net 27 GNDA))
     (model ${KISYS3DMOD}/TestPoint.3dshapes/TestPoint_Keystone_5000-5004_Miniature.wrl
       (at (xyz 0 0 0))
@@
       (effects (font (size 0.75 0.75) (thickness 0.1)))
     )
-    (fp_text value 1uF (at 0 1.17) (layer F.Fab)
+    (fp_text value 10uF (at 0 1.17) (layer F.Fab)
       (effects (font (size 1 1) (thickness 0.15)))
     )
@@
       (effects (font (size 0.75 0.75) (thickness 0.1)))
     )
-    (fp_text value 1uF (at 0 1.17) (layer F.Fab)
-      (effects (font (size 1 1) (thickness 0.15)))
-    )
+    (fp_text value 10uF (at 0 1.17) (layer F.Fab)
+      (effects (font (size 1 1) (thickness 0.15)))
+    )
