File: Technology/ESLO_RB/ESLO_RB.sch (KiCad schematic (older format))
At the start: 71 parts, among them J1 Board to Board, J2 Conn_01x10_Female, U1 TPS62740, U10 MT29F2G01ABBGDWB-IT:G TR, U2 LP5907MFX-1.5, U3 CC2652RB, U4 2450BM14G0011, U5 MAX1720, U6 TPS72301DDCT, U7 ADS1294, U8 LSM303AGR, U9 CY15V104QI-20LPXC

Commit message: Redo ESLO_RB with AC coupling
Parts:
- removed C25, C27, C28: 4.7nF, Capacitor_SMD:C_0402_1005Metric, symbol Device:C
- removed C26: 1000pF, Capacitor_SMD:C_0402_1005Metric, symbol Device:C
- removed R12, R14, R15, R16, R17, R18: 4.7k, Resistor_SMD:R_0402_1005Metric, symbol Device:R
- removed R13: 1M, Resistor_SMD:R_0402_1005Metric, symbol Device:R
- added CN3, CN7: 1000pF, ARBO Parts:0508_array, symbol ARBO_library:C_Pack04
- added CN4, CN8: 1uF, ARBO Parts:0508_array, symbol ARBO_library:C_Pack04
- added CN9: 4700pF, ARBO Parts:0508_array, symbol ARBO_library:C_Pack04
- added RN1, RN5: 4.7k, ARBO Parts:0502_array, symbol Device:R_Pack04
- added RN2, RN6: 1M, ARBO Parts:0502_array, symbol Device:R_Pack04
- renumbered C9 to C10, C10 to C11, C13 to C12, C14 to C13, C16 to C14, C17 to C15, C18 to C16, C19 to C17, C20 to C18, C21 to C19, C22 to C20, C23 to C21, C29 to C26, C30 to C27, C31 to C28, C32 to C29, C33 to C30, C34 to C31, C35 to C32, C36 to C33, C37 to C34, C38 to C35, C39 to C36, C11 to C8, C8 to C9, R7 to R11, R8 to R7, R9 to R8
Connections:
- net EEG_SCK is gone; now on net EEG_SCLK: U7.8F (SCLK)
- net FRAM_CS is gone; now on net _FRAM_CS: U9.1 (~CS)
- net INT1_XL is gone; now on net AXY_INT1: U8.12 (INT1_XL)
- net INT2_XL is gone; now on net AXY_INT2: U8.11 (INT2_XL)
- net MAG_INT is gone; now on net _AXY_MAG: U8.7 (INT_MAG/DRDY)
- net NAND_CS is gone; now on net _NAND_CS: U10.1 (~CS)
- net AXY_INT1: now also U3.18 (DIO_12)
- net DEBUG: now also U3.20 (DIO_14)
- net EEG_MISO: now also U3.27 (DIO_17); no longer U3.14 (DIO_8)
- net EEG_MOSI: now also U3.28 (DIO_18); no longer U3.15 (DIO_9)
- net EEG_SCLK: now also U3.29 (DIO_19); no longer U3.16 (DIO_10)
- net EEG_START: now also U3.32 (DIO_22)
- net GNDA: now also J2.8 (Pin_8); no longer C18.1, C19.1
- net GNDD: now also C18.1, C19.1
- net MISO: now also U3.14 (DIO_8)
- net MOSI: now also U3.15 (DIO_9)
- net R_VBATT: now also U3.38 (DIO_25); no longer U3.36 (DIO_23)
- net VSSA: now also CN7.5 (C4.2), CN7.6 (C3.2), CN7.7 (C2.2), CN7.8 (C1.2)
- net _EEG_CS: now also U3.31 (DIO_21)
- net _EEG_DRDY: now also U3.36 (DIO_23)
- net _FRAM_CS: now also U3.17 (DIO_11)
- net _NAND_CS: now also U3.30 (DIO_20)
- net _SHDN: now also U3.11 (DIO_6)
- net ~SHDN: now also U3.26 (DIO_16)
- net at U7.1E (IN4P): now also CN4.8 (C1.2), RN2.1 (R1.1)
- net at U7.1F (IN3P): now also CN4.6 (C3.2), RN2.3 (R3.1)
- net at U7.1G (IN2P): now also CN8.8 (C1.2), RN6.1 (R1.1)
- net at U7.1H (IN1P): now also CN8.6 (C3.2), RN6.3 (R3.1)
- net at U7.2E (IN4N): now also CN4.7 (C2.2), RN2.2 (R2.1)
- net at U7.2F (IN3N): now also CN4.5 (C4.2), RN2.4 (R4.1)
- net at U7.2G (IN2N): now also CN8.7 (C2.2), RN6.2 (R2.1)
- net at U7.2H (IN1N): now also CN8.5 (C4.2), RN6.4 (R4.1)
- net at U7.3C (RLDINV): now also U7.3B (RLDOUT), RN2.5 (R4.2), RN2.6 (R3.2), RN2.7 (R2.2), RN2.8 (R1.2), RN6.5 (R4.2), RN6.6 (R3.2), RN6.7 (R2.2), RN6.8 (R1.2)
- net AXY_INT2: now reaches U3.19 (DIO_13)
- net SCK renamed SCLK
- net SCLK: now also U3.16 (DIO_10)
- new net: CN3.4 (C4.1), CN4.4 (C4.1), CN9.7 (C2.2), RN1.5 (R4.2)
- new net: CN3.3 (C3.1), CN4.3 (C3.1), CN9.2 (C2.1), RN1.6 (R3.2)
- new net: CN3.2 (C2.1), CN4.2 (C2.1), CN9.1 (C1.1), RN1.7 (R2.2)
- new net: CN3.1 (C1.1), CN4.1 (C1.1), CN9.8 (C1.2), RN1.8 (R1.2)
- new net: CN7.1 (C1.1), CN8.1 (C1.1), CN9.3 (C3.1), RN5.8 (R1.2)
- new net: CN7.3 (C3.1), CN8.3 (C3.1), CN9.4 (C4.1), RN5.6 (R3.2)
- new net: CN7.4 (C4.1), CN8.4 (C4.1), CN9.5 (C4.2), RN5.5 (R4.2)
- new net: CN7.2 (C2.1), CN8.2 (C2.1), CN9.6 (C3.2), RN5.7 (R2.2)
- now unconnected: J2.7 (Pin_7), U7.3A (RLDIN)
- no-connect marks 13 -> 18
Other:
- note added: "BTN1\nBTN2"
- note added: "RD LED\nGR LED\nSPI\nSPI\nSPI"
- note added: "UART\nUART"
- note removed: "ADC\nADC"
- note removed: "GR LED\nSPI\nSPI\nSPI"
- moved on the sheet: J2, R11

Commit message: Completed RB design
Parts:
- removed C18, C28: 1uF, Capacitor_SMD:C_0402_1005Metric, symbol Device:C
- removed C27: 10uF, Capacitor_SMD:C_0603_1608Metric, symbol Device:C
- removed R1: 4.7k, Resistor_SMD:R_0402_1005Metric, symbol Device:R
Connections:
- net +1V8: no longer R2.1, R3.1
- net GNDA: no longer J2.8 (Pin_8)
- net GNDD: now also D1.1 (K)
- net VDD: now also R2.1, R3.1
- net VDDA: now also U7.3A (RLDIN)
- net VSSA: now also CN3.5 (C4.2), CN3.6 (C3.2), CN3.7 (C2.2), CN3.8 (C1.2)
- net at J2.1 (Pin_1): now also RN5.4 (R4.1)
- net at J2.2 (Pin_2): now also RN5.3 (R3.1)
- net at J2.3 (Pin_3): now also RN5.2 (R2.1)
- net at J2.4 (Pin_4): now also RN5.1 (R1.1)
- net at J2.5 (Pin_5): now also RN1.4 (R4.1)
- net at J2.6 (Pin_6): now also RN1.3 (R3.1)
- net at J2.7 (Pin_7): now also RN1.2 (R2.1)
- net at RN1.1 (R1.1): now also J2.8 (Pin_8)
- no-connect marks 18 -> 17
Other:
- note added: "LED is 3v, no R"
- note added: "SHARED 2.2uF replaces 1uF"
- note added: "SHARED CAP"
- note added: "SHARED caps on VDD\nthis remains ‘local’"
- note added: "Shared 1uF cap"
- note added: "or GNDD"
- note removed: "CAP ON EEG"
- moved on the sheet: C16, C26, C29, D1, J2, R11, R2, R3

Commit message: Checked all pins, ready for production
Parts:
- AE1: value Antenna -> 2450AT42B100
- L3: Digikey (none) -> 712-1416-1-ND
- L4: Digikey (none) -> 712-1411-1-ND
Connections:
- net EEG_CS is gone; now on net _EEG_CS: U7.7F (~CS)
- net EEG_DRDY is gone; now on net _EEG_DRDY: U7.6D (~DRDY)
- net DEBUG renamed _DEBUG
- net _AXY_CS: no longer names the net of U3.9 (DIO_4)
- net _SHDN: no longer names the net of U3.11 (DIO_6)
- no-connect marks 17 -> 18
Other:
- note added: "LOW for DEBUG mode"
- note added: "Use int pull-up"
Changed lines of the file:
@@
 L power:GNDD #PWR039
 U 1 1 5F61C685
-P 14800 8450
-F 0 "#PWR039" H 14800 8200 50  0001 C CNN
-F 1 "GNDD" H 14804 8295 50  0000 C CNN
-F 2 "" H 14800 8450 50  0001 C CNN
-F 3 "" H 14800 8450 50  0001 C CNN
-	1    14800 8450
-	1    0    0    -1
-$EndComp
-Connection ~ 14800 8450
+P 15300 8450
+F 0 "#PWR039" H 15300 8200 50  0001 C CNN
+F 1 "GNDD" H 15304 8295 50  0000 C CNN
+F 2 "" H 15300 8450 50  0001 C CNN
+F 3 "" H 15300 8450 50  0001 C CNN
+	1    15300 8450
+	1    0    0    -1
+$EndComp
 NoConn ~ 14800 7850
 $Comp
@@
 EEG_START
 Text GLabel 13000 7950 0    50   Input ~ 0
-EEG_CS
+_EEG_CS
 Text GLabel 13000 8050 0    50   Input ~ 0
-EEG_DRDY
+_EEG_DRDY
 Text GLabel 13000 8250 0    50   Input ~ 0
 EEG_MOSI
@@
 P 14950 2950
 F 0 "AE1" H 15030 2939 50  0000 L CNN
-F 1 "Antenna" H 15030 2848 50  0000 L CNN
+F 1 "2450AT42B100" H 15030 2848 50  0000 L CNN
 F 2 "ARBO Parts:2450AT42B100" H 14950 2950 50  0001 C CNN
 F 3 "~" H 14950 2950 50  0001 C CNN
@@
 	11150 3550 11750 3550
 Text GLabel 11150 3950 2    50   Input ~ 0
-DEBUG
+_DEBUG
 Text GLabel 12500 3050 0    50   Input ~ 0
 EEG_SCLK
@@
 Text GLabel 12500 3550 0    50   Input ~ 0
 THERM
-Text GLabel 12500 1750 0    50   Input ~ 0
-_SHDN
 Text GLabel 12500 2250 0    50   Input ~ 0
 _FRAM_CS
@@
 Text GLabel 12500 3450 0    50   Input ~ 0
 _EEG_DRDY
-Text GLabel 12500 1550 0    50   Input ~ 0
-_AXY_CS
 Text GLabel 12500 1650 0    50   Input ~ 0
 _AXY_MAG
@@
 AXY_INT2
 Text GLabel 12500 2550 0    50   Input ~ 0
-DEBUG
+_DEBUG
 Text GLabel 12500 3650 0    50   Input ~ 0
 R_VBATT
@@
 F 2 "Inductor_SMD:L_0402_1005Metric" H 14800 3150 50  0001 C CNN
 F 3 "~" H 14800 3150 50  0001 C CNN
+F 4 "712-1416-1-ND" H 14800 3150 50  0001 C CNN "Digikey"
 	1    14800 3150
 	0    -1   -1   0
@@
 F 2 "Inductor_SMD:L_0402_1005Metric" H 14650 3300 50  0001 C CNN
 F 3 "~" H 14650 3300 50  0001 C CNN
+F 4 "712-1411-1-ND" H 14650 3300 50  0001 C CNN "Digikey"
 	1    14650 3300
 	1    0    0    -1
@@
 NoConn ~ 12500 4050
 NoConn ~ 15750 2450
-NoConn ~ 4300 1700
 Text GLabel 12500 2750 0    50   Input ~ 0
 ~SHDN
@@
 or GNDD
 $Comp
-L power:VDD #PWR?
+L power:VDD #PWR0105
 U 1 1 600DAA35
 P 4500 8550
-F 0 "#PWR?" H 4500 8400 50  0001 C CNN
+F 0 "#PWR0105" H 4500 8400 50  0001 C CNN
 F 1 "VDD" H 4517 8723 50  0000 C CNN
 F 2 "" H 4500 8550 50  0001 C CNN
@@
 $EndComp
 $Comp
-L power:VDD #PWR?
+L power:VDD #PWR0106
 U 1 1 600DADB1
 P 4200 8550
-F 0 "#PWR?" H 4200 8400 50  0001 C CNN
+F 0 "#PWR0106" H 4200 8400 50  0001 C CNN
 F 1 "VDD" H 4217 8723 50  0000 C CNN
 F 2 "" H 4200 8550 50  0001 C CNN
@@
 	1    0    0    -1
 $EndComp
+NoConn ~ 12500 1750
+Connection ~ 15300 8450
+NoConn ~ 12500 1550
+Text Notes 11600 2600 0    50   ~ 0
+Use int pull-up
+Text Notes 11150 4100 0    50   ~ 0
+LOW for DEBUG mode
 $EndSCHEMATC

Commit message: Submit ESLO_RB for mfg w PCBONLINE
Parts:
- C1: Digikey 490-3896-1-ND -> 1276-2868-1-ND
- C10: renamed from C15; Digikey 490-6326-2-ND -> 1276-1051-1-ND
- C11: renamed from C7; value 100nF -> 0.1uF; Digikey 490-6319-1-ND -> 490-6328-1-ND
- C12: renamed from C14; Digikey 490-12532-1-ND -> 1276-1469-1-ND
- C19: renamed from C36; Digikey 490-6350-2-ND -> 478-1101-1-ND
- C2: renamed from C12; Digikey 490-3896-1-ND -> 1276-2868-1-ND
- C22: renamed from C10; value 100nF -> 0.1uF; Digikey 490-6319-1-ND -> 490-6328-1-ND
- C25: renamed from C9; value 100nF -> 0.1uF; Digikey 490-6319-1-ND -> 490-6328-1-ND
- C26: renamed from C6; value 100nF -> 0.1uF; Digikey 490-6319-1-ND -> 490-6328-1-ND
- C28: renamed from C5; value 100nF -> 0.1uF; Digikey 490-6319-1-ND -> 490-6328-1-ND
- C29: renamed from C4; value 100nF -> 0.1uF; Digikey 490-6319-1-ND -> 490-6328-1-ND
- C4: renamed from C13; Digikey 490-3896-1-ND -> 1276-2868-1-ND
- C6: renamed from C2; Digikey 490-3896-1-ND -> 1276-2868-1-ND
- C7: renamed from C30; value 220nF -> 0.22uF; Digikey 490-14372-1-ND -> 1276-1176-1-ND
- C8: renamed from C3; Digikey 490-12532-1-ND -> 1276-1469-1-ND
- D1: Digikey 732-4971-1-ND -> SML-D12V1WT86CT-ND
- J1: renamed from J2; value Conn_01x10_Female -> 10POS Biopotentials; Digikey H125102CT-ND -> ED10276-ND
- J2: renamed from J1; value Board to Board -> 6POS Power/JTAG; Digikey H125100CT-ND -> ED10273-ND
- renumbered C31 to C13, C32 to C14, C33 to C15, C34 to C16, C35 to C18, C19 to C20, C11 to C21, C29 to C23, C20 to C24, C21 to C27, C26 to C3, C8 to C5, C16 to C9, CN9 to CN1, CN3 to CN2, CN7 to CN3, CN8 to CN5, L4 to L3, L3 to L4, R4 to R1, R6 to R2, R5 to R3, R7 to R4, R8 to R5, R2 to R6, R3 to R7, R11 to R8, RN5 to RN2, RN2 to RN3, RN6 to RN4, U5 to U1, U4 to U10, U1 to U2, U9 to U3, U8 to U4, U2 to U5, U10 to U7, U3 to U8, U7 to U9
Other:
- note added: "!!Needs 1.8V for level shifters"
- note removed: "Can HOLD and WP float?"
- moved on the sheet: C11, C3, C7, D1, R1, R2, R3, R6, R7, U3, U4, U7

Commit message: Debugger submitted
Parts:
- C1, C2, C4, C6: Digikey 1276-2868-1-ND -> 490-14372-1-ND
Changed lines of the file:
@@
 F 2 "Capacitor_SMD:C_0603_1608Metric" H 2638 1000 50  0001 C CNN
 F 3 "~" H 2600 1150 50  0001 C CNN
-F 4 "1276-2868-1-ND" H 2600 1150 50  0001 C CNN "Digikey"
+F 4 "490-14372-1-ND" H 2600 1150 50  0001 C CNN "Digikey"
 	1    2600 1150
 	1    0    0    1
@@
 F 2 "Capacitor_SMD:C_0603_1608Metric" H 988 1000 50  0001 C CNN
 F 3 "~" H 950 1150 50  0001 C CNN
-F 4 "1276-2868-1-ND" H 950 1150 50  0001 C CNN "Digikey"
+F 4 "490-14372-1-ND" H 950 1150 50  0001 C CNN "Digikey"
 	1    950  1150
 	1    0    0    1
@@
 F 2 "Capacitor_SMD:C_0603_1608Metric" H 1438 3000 50  0001 C CNN
 F 3 "~" H 1400 3150 50  0001 C CNN
-F 4 "1276-2868-1-ND" H 1400 3150 50  0001 C CNN "Digikey"
+F 4 "490-14372-1-ND" H 1400 3150 50  0001 C CNN "Digikey"
 	1    1400 3150
 	0    -1   1    0
@@
 F 2 "Capacitor_SMD:C_0603_1608Metric" H 2388 3450 50  0001 C CNN
 F 3 "~" H 2350 3600 50  0001 C CNN
-F 4 "1276-2868-1-ND" H 2350 3600 50  0001 C CNN "Digikey"
+F 4 "490-14372-1-ND" H 2350 3600 50  0001 C CNN "Digikey"
 	1    2350 3600
 	-1   0    0    -1

Commit message: Assembling ESLO_RB
Parts:
- AE1: Digikey 712-1600-1-ND -> 712-1008-1-ND‎
Connections:
- net RESET_N is gone; now on net _RESET: U2.7 (PG)
Other:
- note added: "(-1.8v)"
- note added: "10nF = 10000pF"
- note removed: "(-3v)"
Changed lines of the file:
@@
 	1550 3150 1550 3250
 Text Notes 2400 3400 2    50   ~ 0
-(-3v)
+(-1.8v)
 $Comp
 L power:VDDA #PWR022
@@
 F 2 "ARBO Parts:2450AT42B100" H 14950 2950 50  0001 C CNN
 F 3 "~" H 14950 2950 50  0001 C CNN
-F 4 "712-1600-1-ND" H 14950 2950 50  0001 C CNN "Digikey"
+F 4 "712-1008-1-ND‎" H 14950 2950 50  0001 C CNN "Digikey"
 	1    14950 2950
 	1    0    0    -1
@@
 SCLK
 Text GLabel 2050 1400 2    50   Input ~ 0
-RESET_N
+_RESET
 Wire Wire Line
 	2600 1300 3450 1300
@@
 Text Notes 9750 4000 0    50   ~ 0
 !!Needs 1.8V for level shifters
+Text Notes 3450 4200 0    50   ~ 0
+10nF = 10000pF
 $EndSCHEMATC
