File: Technology/ESLO_COIN_POWER/ESLO_COIN_POWER.kicad_pcb (KiCad board)
At the start: 2 copper layers, 46.8 x 35.5 mm, 3 parts, among them J1 Conn_02x03_Counter_Clockwise

Commit message: Schematics
Parts:
- J1: moved to B.Cu
- moved J1 2.50 mm to (74.8, 97.8), turned to 270 degrees
Connections:
- J1 pad 1: (no net) -> GND
- J1 pad 2: GND -> (no net)
- J1 pad 5: (no net) -> Net-(BT1-Pad1)
- J1 pad 6: Net-(BT1-Pad1) -> (no net)
Changed lines of the file:
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@@
     (add_net "Net-(BT1-Pad1)")
   )
-  (module Connector_PinSocket_2.54mm:PinSocket_2x03_P2.54mm_Vertical (layer F.Cu)
-    (at 74.75 95.25 90)
+  (module Connector_PinSocket_2.54mm:PinSocket_2x03_P2.54mm_Vertical (layer B.Cu)
+    (at 74.75 97.75 270)
     (descr "Through hole straight socket strip, 2x03, 2.54mm pitch, double cols (from Kicad 4.0.7), script generated")
     (tags "Through hole socket strip THT 2x03 2.54mm double row")
-    (fp_text reference J1 (at -3.75 8 180) (layer F.SilkS)
-      (effects (font (size 1 1) (thickness 0.15)))
+    (fp_text reference J1 (at -3.75 -8 180) (layer B.SilkS)
+      (effects (font (size 1 1) (thickness 0.15)) (justify mirror))
     )
-    (fp_text value Conn_02x03_Counter_Clockwise (at -1.27 7.85 90) (layer F.Fab)
-      (effects (font (size 1 1) (thickness 0.15)))
+    (fp_text value Conn_02x03_Counter_Clockwise (at -1.27 -7.85 270) (layer B.Fab)
+      (effects (font (size 1 1) (thickness 0.15)) (justify mirror))
     )
-    (fp_text user %R (at -1.27 2.54) (layer F.Fab)
-      (effects (font (size 1 1) (thickness 0.15)))
+    (fp_text user %R (at -1.27 -2.54) (layer B.Fab)
+      (effects (font (size 1 1) (thickness 0.15)) (justify mirror))
     )
-    (fp_line (start -4.34 6.85) (end -4.34 -1.8) (layer F.CrtYd) (width 0.05))
-    (fp_line (start 1.76 6.85) (end -4.34 6.85) (layer F.CrtYd) (width 0.05))
-    (fp_line (start 1.76 -1.8) (end 1.76 6.85) (layer F.CrtYd) (width 0.05))
-    (fp_line (start -4.34 -1.8) (end 1.76 -1.8) (layer F.CrtYd) (width 0.05))
-    (fp_line (start 0 -1.33) (end 1.33 -1.33) (layer F.SilkS) (width 0.12))
-    (fp_line (start 1.33 -1.33) (end 1.33 0) (layer F.SilkS) (width 0.12))
-    (fp_line (start -1.27 -1.33) (end -1.27 1.27) (layer F.SilkS) (width 0.12))
-    (fp_line (start -1.27 1.27) (end 1.33 1.27) (layer F.SilkS) (width 0.12))
-    (fp_line (start 1.33 1.27) (end 1.33 6.41) (layer F.SilkS) (width 0.12))
-    (fp_line (start -3.87 6.41) (end 1.33 6.41) (layer F.SilkS) (width 0.12))
-    (fp_line (start -3.87 -1.33) (end -3.87 6.41) (layer F.SilkS) (width 0.12))
-    (fp_line (start -3.87 -1.33) (end -1.27 -1.33) (layer F.SilkS) (width 0.12))
-    (fp_line (start -3.81 6.35) (end -3.81 -1.27) (layer F.Fab) (width 0.1))
-    (fp_line (start 1.27 6.35) (end -3.81 6.35) (layer F.Fab) (width 0.1))
-    (fp_line (start 1.27 -0.27) (end 1.27 6.35) (layer F.Fab) (width 0.1))
-    (fp_line (start 0.27 -1.27) (end 1.27 -0.27) (layer F.Fab) (width 0.1))
-    (fp_line (start -3.81 -1.27) (end 0.27 -1.27) (layer F.Fab) (width 0.1))
-    (pad 6 thru_hole oval (at -2.54 5.08 90) (size 1.7 1.7) (drill 1) (layers *.Cu *.Mask)
+    (fp_line (start -4.34 -6.85) (end -4.34 1.8) (layer B.CrtYd) (width 0.05))
+    (fp_line (start 1.76 -6.85) (end -4.34 -6.85) (layer B.CrtYd) (width 0.05))
+    (fp_line (start 1.76 1.8) (end 1.76 -6.85) (layer B.CrtYd) (width 0.05))
+    (fp_line (start -4.34 1.8) (end 1.76 1.8) (layer B.CrtYd) (width 0.05))
+    (fp_line (start 0 1.33) (end 1.33 1.33) (layer B.SilkS) (width 0.12))
+    (fp_line (start 1.33 1.33) (end 1.33 0) (layer B.SilkS) (width 0.12))
+    (fp_line (start -1.27 1.33) (end -1.27 -1.27) (layer B.SilkS) (width 0.12))
+    (fp_line (start -1.27 -1.27) (end 1.33 -1.27) (layer B.SilkS) (width 0.12))
+    (fp_line (start 1.33 -1.27) (end 1.33 -6.41) (layer B.SilkS) (width 0.12))
+    (fp_line (start -3.87 -6.41) (end 1.33 -6.41) (layer B.SilkS) (width 0.12))
+    (fp_line (start -3.87 1.33) (end -3.87 -6.41) (layer B.SilkS) (width 0.12))
+    (fp_line (start -3.87 1.33) (end -1.27 1.33) (layer B.SilkS) (width 0.12))
+    (fp_line (start -3.81 -6.35) (end -3.81 1.27) (layer B.Fab) (width 0.1))
+    (fp_line (start 1.27 -6.35) (end -3.81 -6.35) (layer B.Fab) (width 0.1))
+    (fp_line (start 1.27 0.27) (end 1.27 -6.35) (layer B.Fab) (width 0.1))
+    (fp_line (start 0.27 1.27) (end 1.27 0.27) (layer B.Fab) (width 0.1))
+    (fp_line (start -3.81 1.27) (end 0.27 1.27) (layer B.Fab) (width 0.1))
+    (pad 6 thru_hole oval (at -2.54 -5.08 270) (size 1.7 1.7) (drill 1) (layers *.Cu *.Mask))
+    (pad 5 thru_hole oval (at 0 -5.08 270) (size 1.7 1.7) (drill 1) (layers *.Cu *.Mask)
       (net 2 "Net-(BT1-Pad1)"))
-    (pad 5 thru_hole oval (at 0 5.08 90) (size 1.7 1.7) (drill 1) (layers *.Cu *.Mask))
-    (pad 4 thru_hole oval (at -2.54 2.54 90) (size 1.7 1.7) (drill 1) (layers *.Cu *.Mask))
-    (pad 3 thru_hole oval (at 0 2.54 90) (size 1.7 1.7) (drill 1) (layers *.Cu *.Mask))
-    (pad 2 thru_hole oval (at -2.54 0 90) (size 1.7 1.7) (drill 1) (layers *.Cu *.Mask)
+    (pad 4 thru_hole oval (at -2.54 -2.54 270) (size 1.7 1.7) (drill 1) (layers *.Cu *.Mask))
+    (pad 3 thru_hole oval (at 0 -2.54 270) (size 1.7 1.7) (drill 1) (layers *.Cu *.Mask))
+    (pad 2 thru_hole oval (at -2.54 0 270) (size 1.7 1.7) (drill 1) (layers *.Cu *.Mask))
+    (pad 1 thru_hole rect (at 0 0 270) (size 1.7 1.7) (drill 1) (layers *.Cu *.Mask)
       (net 1 GND))
-    (pad 1 thru_hole rect (at 0 0 90) (size 1.7 1.7) (drill 1) (layers *.Cu *.Mask))
     (model ${KISYS3DMOD}/Connector_PinSocket_2.54mm.3dshapes/PinSocket_2x03_P2.54mm_Vertical.wrl
       (at (xyz 0 0 0))
