File: Technology/ESLO_COIN_POWER/ESLO_COIN_POWER.sch (KiCad schematic (older format))
At the start: 3 parts, among them J1 Conn_02x03_Counter_Clockwise

Commit message: Schematics
Connections:
- net GND: now also J1.1 (Pin_1); no longer J1.2 (Pin_2)
- net at J1.5 (Pin_5): now also BT1.1 (+), BT2.1 (+)
- now unconnected: J1.6 (Pin_6)
Changed lines of the file:
@@
 L Connector_Generic:Conn_02x03_Odd_Even J1
 U 1 1 60BE1518
-P 3550 1100
-F 0 "J1" H 3600 1417 50  0000 C CNN
-F 1 "Conn_02x03_Counter_Clockwise" H 3600 1326 50  0000 C CNN
-F 2 "Connector_PinSocket_2.54mm:PinSocket_2x03_P2.54mm_Vertical" H 3550 1100 50  0001 C CNN
-F 3 "~" H 3550 1100 50  0001 C CNN
-F 4 "A106656-ND" H 3550 1100 50  0001 C CNN "Digikey"
-	1    3550 1100
-	-1   0    0    1
+P 3450 1100
+F 0 "J1" H 3450 900 50  0000 C CNN
+F 1 "Conn_02x03_Counter_Clockwise" H 3900 1300 50  0000 C CNN
+F 2 "Connector_PinSocket_2.54mm:PinSocket_2x03_P2.54mm_Vertical" H 3450 1100 50  0001 C CNN
+F 3 "~" H 3450 1100 50  0001 C CNN
+F 4 "A106656-ND" H 3450 1100 50  0001 C CNN "Digikey"
+	1    3450 1100
+	1    0    0    1
 $EndComp
 $Comp
@@
 	1    0    0    -1
 $EndComp
-Connection ~ 3250 1200
 Wire Wire Line
 	3250 1000 2900 1000
@@
 NoConn ~ 3750 1200
 NoConn ~ 3250 1100
+Connection ~ 3250 1200
 $EndSCHEMATC
