File: Technology/ESLO_RB2/ESLO_RB2.sch (KiCad schematic (older format))
At the start: 68 parts, among them CN1 4700pF, CN2 1000pF, CN3 1000pF, CN4 0.1uF, CN5 0.1uF, J1 Biopotentials, J2 PWR/COMM, J3 Conn_01x02_Female, U1 MAX1720, U10 2450BM14G0011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

Commit message: Schematics
Other:
- note added: "Need to be careful about shared caps, can lead to unstable power supplies"
- note added: "This PCB layout needs work, see datasheet and reference design"
Changed lines of the file:
@@
 Text Notes 12450 2250 0    50   ~ 0
 Use 0603 for compatability with BAW version (reqs 10uF)
+Text Notes 2200 1700 0    50   ~ 0
+This PCB layout needs work, see datasheet and reference design
+Text Notes 350  350  0    50   ~ 0
+Need to be careful about shared caps, can lead to unstable power supplies
 $EndSCHEMATC

Commit message: Comments
Other:
- note added: "This PCB layout needs work (there’s a power pad!), see datasheet and reference design"
- note removed: "This PCB layout needs work, see datasheet and reference design"
Changed lines of the file:
@@
 Use 0603 for compatability with BAW version (reqs 10uF)
 Text Notes 2200 1700 0    50   ~ 0
-This PCB layout needs work, see datasheet and reference design
+This PCB layout needs work (there’s a power pad!), see datasheet and reference design
 Text Notes 350  350  0    50   ~ 0
 Need to be careful about shared caps, can lead to unstable power supplies

Commit message: Update schematics
Other:
- note added: "BTN1"
- note added: "Use int pull-up, BTN2"
- note removed: "BTN1\nBTN2"
- note removed: "Use int pull-up"
Changed lines of the file:
@@
 SHARED CAP
 Text Notes 10450 2500 0    50   ~ 0
-BTN1\nBTN2
+BTN1
 Text GLabel 11050 2150 0    50   Input ~ 0
 SCLK
@@
 Connection ~ 15300 8450
 NoConn ~ 11050 1550
-Text Notes 10100 2600 0    50   ~ 0
-Use int pull-up
+Text Notes 9850 2600 0    50   ~ 0
+Use int pull-up, BTN2
 Text Notes 7450 4300 0    50   ~ 0
 LOW for DEBUG mode\nUse ED8250-ND 50-pos pins to interface
