File: Technology/ESLO_RB2_DataDump/ESLO_RB2_DataDump.sch (KiCad schematic (older format))
At the start: 12 parts, among them J1 Conn_01x08_Female, SW1 SW_DPST, U1 TPS62243_WSON, U2 Adalogger, U3 SN74ACX1T45, U4 SN74ACX1T45

Commit message: Schematics
Other:
- note added: "!! Add input cap, this design will fail"
- note removed: "No cap needed, 3.3V is regulated on Adalogger"
Changed lines of the file:
@@
 Connection ~ 1300 1900
 Text Notes 1150 1100 0    50   ~ 0
-No cap needed, 3.3V is regulated on Adalogger
+!! Add input cap, this design will fail
 $EndSCHEMATC

Commit message: Update schematics
Connections:
- net +1V8: no longer J1.4 (Pin_4)
- net +3V3: now also J1.4 (Pin_4)
Other:
- note added: "!!changed to 3.3V from 1.8V\nmistake on PCB"
Changed lines of the file:
@@
 DEBUG
-$Comp
-L power:+1V8 #PWR0104
-U 1 1 60BAD4A6
-P 1550 2900
-F 0 "#PWR0104" H 1550 2750 50  0001 C CNN
-F 1 "+1V8" H 1565 3073 50  0000 C CNN
-F 2 "" H 1550 2900 50  0001 C CNN
-F 3 "" H 1550 2900 50  0001 C CNN
-	1    1550 2900
-	1    0    0    -1
-$EndComp
 $Comp
 L power:GND #PWR0105
@@
 Text Notes 1150 1100 0    50   ~ 0
 !! Add input cap, this design will fail
+Text Notes 900  3000 2    50   ~ 0
+!!changed to 3.3V from 1.8V\nmistake on PCB
+$Comp
+L power:+3V3 #PWR?
+U 1 1 60F1A17C
+P 1550 2900
+F 0 "#PWR?" H 1550 2750 50  0001 C CNN
+F 1 "+3V3" H 1565 3073 50  0000 C CNN
+F 2 "" H 1550 2900 50  0001 C CNN
+F 3 "" H 1550 2900 50  0001 C CNN
+	1    1550 2900
+	1    0    0    -1
+$EndComp
 $EndSCHEMATC
